Commit message: new commit

File: description/robot_core.xacro (robot description, xacro)
@@ -41,9 +41,12 @@
         </xacro:inertial_box>
     </link>
+    <gazebo reference="chassis">
+        <material>Gazebo/Orange</material>
+    </gazebo>
     <!-- LEFT WHEEL LINK -->
     <joint name="left_wheel_joint" type="continuous">
         <parent link="base_link"/>
         <child link="left_wheel"/>
-        <origin xyz="0 0.2 0.05" rpy="-${pi/2} 0 0"/>
+        <origin xyz="0 0.22 0.05" rpy="-${pi/2} 0 0"/>
         <axis xyz="0 0 1"/>
     </joint>
@@ -64,9 +67,12 @@
         </xacro:inertial_cylinder>
     </link>
+    <gazebo reference="left_wheel">
+        <material>Gazebo/Black</material>
+    </gazebo>
     <!-- RIGHT WHEEL LINK -->
     <joint name="right_wheel_joint" type="continuous">
         <parent link="base_link"/>
         <child link="right_wheel"/>
-        <origin xyz="0 -0.2 0.05" rpy="${pi/2} 0 0"/>
+        <origin xyz="0 -0.22 0.05" rpy="${pi/2} 0 0"/>
         <axis xyz="0 0 -1"/>
     </joint>
@@ -87,7 +93,10 @@
         </xacro:inertial_cylinder>
     </link>
+    <gazebo reference="right_wheel">
+        <material>Gazebo/Black</material>
+    </gazebo>
     <!-- LEFT CASTER WHEEL LINK -->
     <joint name="left_caster_wheel_joint" type="fixed">
-        <parent link="base_link"/>
+        <parent link="chassis"/>
         <child link="left_caster_wheel"/>
         <origin xyz="0.42 0.1 0"/>
@@ -109,7 +118,12 @@
         </xacro:inertial_sphere>
     </link>
+    <gazebo reference="left_caster_wheel">
+        <material>Gazebo/Black</material>
+        <mu1 value="0.001"/>
+        <mu2 value="0.001"/>
+    </gazebo>
     <!-- RIGHT CASTER WHEEL LINK -->
     <joint name="right_caster_wheel_joint" type="fixed">
-        <parent link="base_link"/>
+        <parent link="chassis"/>
         <child link="right_caster_wheel"/>
         <origin xyz="0.42 -0.1 0"/>
@@ -131,3 +145,8 @@
         </xacro:inertial_sphere>
     </link>
+    <gazebo reference="right_caster_wheel">
+        <material>Gazebo/Black</material>
+        <mu1 value="0.001"/>
+        <mu2 value="0.001"/>
+    </gazebo>
 </robot>
